File: tastatur/keyboard-layout/vz200-keyboard-layout.kicad_pcb (KiCad board)
At the start: 2 copper layers, 174.5 x 71.6 mm, 48 parts, among them P1 PWR-LED, SW1 key7, SW10 key-dot, SW11 key9, SW12 key6, SW13 key3, SW14 keyA, SW15 keyF, SW16 keyK, SW17 keyP, SW18 keyU, SW19 keyZ/Y, SW2 key4, SW20 keyB, SW21 keyG, SW22 keyL, SW23 keyQ, SW24 keyV, SW25 key-space, SW26 key-semicolon/Ö, SW27 keyC, SW28 keyH, SW29 keyM, SW3 key1, SW30 keyR, SW31 keyW, SW32 key-apostroph/Ä, SW33 keyD, SW34 keyI, SW35 keyN, SW36 keyS, SW37 keyX, SW38 key-ctrl-left, SW39 key-left-shift, SW4 key-/ß, SW40 keyE, SW41 keyJ, SW42 keyO, SW43 keyT, SW44 keyY/Z, SW45 key-enter, SW5 key-comma, SW6 key8, SW7 key5, SW8 key2, SW9 key0, U1 KeyWarrier24-8Mod

Commit message: Layout Keyboard Platine finalisiert
Parts:
- moved D1 35.2 mm to (244.4, 77.5)
- moved P1 35.2 mm to (156.5, 68.8)
- moved SW10 35.2 mm to (218.9, 117.8)
- moved SW11 35.2 mm to (203.1, 75.8)
- moved SW12 35.2 mm to (163.2, 75.8)
- moved SW15 35.2 mm to (145.8, 103.8)
- moved SW17 35.2 mm to (222.2, 89.8)
- moved SW2 35.2 mm to (136.6, 75.8)
- moved SW21 35.2 mm to (159.1, 103.8)
- moved SW22 35.2 mm to (212.3, 103.8)
- moved SW24 35.2 mm to (152.4, 117.8)
- moved SW25 35.2 mm to (235.5, 117.8)
- moved SW26 35.2 mm to (225.6, 103.8)
- moved SW29 35.2 mm to (192.3, 117.8)
- moved SW3 35.2 mm to (96.7, 75.8)
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Routing:
- net Net-(SW14-Pad2): track 469.7 -> 485.4 mm
- net Net-(SW33-Pad2): track 582.0 -> 597.7 mm
- net Net-(SW39-Pad1): track 259.8 -> 274.2 mm
- net Net-(SW26-Pad1): track 265.5 -> 279.1 mm
- net Net-(SW19-Pad1): track 209.6 -> 219.7 mm
- net Net-(SW10-Pad1): track 640.2 -> 650.0 mm
- net Net-(SW10-Pad2): track 436.3 -> 440.1 mm
- net Net-(SW20-Pad2): track 483.0 -> 486.6 mm
- net Net-(SW1-Pad2): track 521.0 -> 524.1 mm
- net Net-(SW17-Pad1): track 438.8 -> 438.0 mm
Other:
- outline, holes or cut-outs redrawn
