File: tastatur/keyboard-layout/vz200-keyboard-layout.sch (KiCad schematic (older format))
At the start: 48 parts, among them P1 PWR-LED, SW1 key7, SW10 key-dot, SW11 key9, SW12 key6, SW13 key3, SW14 keyA, SW15 keyF, SW16 keyK, SW17 keyP, SW18 keyU, SW19 keyZ/Y, SW2 key4, SW20 keyB, SW21 keyG, SW22 keyL, SW23 keyQ, SW24 keyV, SW25 key-space, SW26 key-semicolon/Ö, SW27 keyC, SW28 keyH, SW29 keyM, SW3 key1, SW30 keyR, SW31 keyW, SW32 key-apostroph/Ä, SW33 keyD, SW34 keyI, SW35 keyN, SW36 keyS, SW37 keyX, SW38 key-ctrl-left, SW39 key-left-shift, SW4 key-/ß, SW40 keyE, SW41 keyJ, SW42 keyO, SW43 keyT, SW44 keyY/Z, SW45 key-enter, SW5 key-comma, SW6 key8, SW7 key5, SW8 key2, SW9 key0, U1 KeyWarrier24-8Mod

Commit message: tastatur /emulator: Reset-Taste (ESC) implementiert; Platinenlayout ergänzt und beschriftet
Parts:
- added P2: Reset-Button, Pin_Headers:Pin_Header_Straight_1x02_Pitch2.54mm, symbol CONN_01X02
- added R1: 110, Resistors_ThroughHole:R_Axial_DIN0204_L3.6mm_D1.6mm_P7.62mm_Horizontal, symbol R
Connections:
- net at SW27.2, SW28.2, SW29.2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: now also P2.1 (P1)
- net at SW39.1, SW45.1, U1.1 (Y0): now also P2.2 (P2)
- net at D1.1 (K): now also R1.2; no longer P1.1 (P1)
- new net: P1.1 (P1), R1.1
Other:
- moved on the sheet: P1
Changed lines of the file:
@@
 	6700 1450 6700 5350
 Wire Wire Line
-	6250 1550 6250 5000
+	6250 1550 6250 5500
 Wire Wire Line
 	6250 1550 3150 1550
@@
 L CONN_01X02 P1
 U 1 1 5CE1B266
-P 7800 2100
-F 0 "P1" H 7800 2250 50  0000 C CNN
-F 1 "PWR-LED" V 7900 2100 50  0000 C CNN
-F 2 "Pin_Headers:Pin_Header_Straight_1x02_Pitch2.54mm" H 7800 2100 50  0001 C CNN
-F 3 "" H 7800 2100 50  0000 C CNN
-	1    7800 2100
+P 7800 1800
+F 0 "P1" H 7800 1950 50  0000 C CNN
+F 1 "PWR-LED" V 7900 1800 50  0000 C CNN
+F 2 "Pin_Headers:Pin_Header_Straight_1x02_Pitch2.54mm" H 7800 1800 50  0001 C CNN
+F 3 "" H 7800 1800 50  0000 C CNN
+	1    7800 1800
 	0    -1   -1   0
 $EndComp
 Wire Wire Line
-	7750 2300 7600 2500
-Wire Wire Line
 	7600 2500 7600 2700
 Wire Wire Line
 	7600 2700 7700 2700
 Wire Wire Line
-	7850 2300 8000 2500
-Wire Wire Line
-	8000 2500 8000 2700
+	8000 2200 8000 2700
 Wire Wire Line
 	8000 2700 7900 2700
+Connection ~ 6050 5150
+Connection ~ 6250 5000
+$Comp
+L R R1
+U 1 1 5D1AA86C
+P 7600 2350
+F 0 "R1" V 7680 2350 50  0000 C CNN
+F 1 "110" V 7600 2350 50  0000 C CNN
+F 2 "Resistors_ThroughHole:R_Axial_DIN0204_L3.6mm_D1.6mm_P7.62mm_Horizontal" V 7530 2350 50  0001 C CNN
+F 3 "" H 7600 2350 50  0000 C CNN
+	1    7600 2350
+	1    0    0    -1
+$EndComp
+Wire Wire Line
+	7600 2200 7750 2000
+Wire Wire Line
+	7850 2000 8000 2200
+$Comp
+L CONN_01X02 P2
+U 1 1 5D1AD3BE
+P 7950 4550
+F 0 "P2" H 7950 4700 50  0000 C CNN
+F 1 "Reset-Button" V 8050 4550 50  0000 C CNN
+F 2 "Pin_Headers:Pin_Header_Straight_1x02_Pitch2.54mm" H 7950 4550 50  0001 C CNN
+F 3 "" H 7950 4550 50  0000 C CNN
+	1    7950 4550
+	0    -1   -1   0
+$EndComp
+Wire Wire Line
+	6250 5500 7900 5500
+Wire Wire Line
+	7900 5500 7900 4750
+Wire Wire Line
+	6050 5150 6050 5600
+Wire Wire Line
+	6050 5600 8000 5600
+Wire Wire Line
+	8000 5600 8000 4750
 $EndSCHEMATC
